Commit message: update

File: ROSManager/urdf/Arm_R.SLDASM.urdf (robot description, URDF)
Before this commit: robot Arm_R.SLDASM, 23 links, 22 joints
Links:
- link FourthFingerArth_1_Link: geometry collision mesh filename=file:///home/yhlmaybe/Documents/Intelligent-Robot-System/RO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; visual mesh filename=file:///home/yhlmaybe/Documents/Intelligent-Robot-System/RO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
- link FourthFingerArth_2_Link: geometry collision mesh filename=file:///home/yhlmaybe/Documents/Intelligent-Robot-System/RO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; visual mesh filename=file:///home/yhlmaybe/Documents/Intelligent-Robot-System/RO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
- link FourthFingerArth_3_Link: geometry collision mesh filename=file:///home/yhlmaybe/Documents/Intelligent-Robot-System/RO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; visual mesh filename=file:///home/yhlmaybe/Documents/Intelligent-Robot-System/RO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
- link FourthFingerArth_4_Link: geometry collision mesh filename=file:///home/yhlmaybe/Documents/Intelligent-Robot-System/RO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; visual mesh filename=file:///home/yhlmaybe/Documents/Intelligent-Robot-System/RO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
- link IndexFingerArth_1_Link: geometry collision mesh filename=file:///home/yhlmaybe/Documents/Intelligent-Robot-System/RO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; visual mesh filename=file:///home/yhlmaybe/Documents/Intelligent-Robot-System/RO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
- link IndexFingerArth_2__Link: geometry collision mesh filename=file:///home/yhlmaybe/Documents/Intelligent-Robot-System/RO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; visual mesh filename=file:///home/yhlmaybe/Documents/Intelligent-Robot-System/RO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
- link IndexFingerArth_3_Link: geometry collision mesh filename=file:///home/yhlmaybe/Documents/Intelligent-Robot-System/RO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; visual mesh filename=file:///home/yhlmaybe/Documents/Intelligent-Robot-System/RO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
- link IndexFingerArth_4_Link: geometry collision mesh filename=file:///home/yhlmaybe/Documents/Intelligent-Robot-System/RO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; visual mesh filename=file:///home/yhlmaybe/Documents/Intelligent-Robot-System/RO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
- link LittleFingerArth_1_Link: geometry collision mesh filename=file:///home/yhlmaybe/Documents/Intelligent-Robot-System/RO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; visual mesh filename=file:///home/yhlmaybe/Documents/Intelligent-Robot-System/RO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
- link LittleFingerArth_2_Link: geometry collision mesh filename=file:///home/yhlmaybe/Documents/Intelligent-Robot-System/RO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; visual mesh filename=file:///home/yhlmaybe/Documents/Intelligent-Robot-System/RO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
- link LittleFingerArth_3_Link: geometry collision mesh filename=file:///home/yhlmaybe/Documents/Intelligent-Robot-System/RO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; visual mesh filename=file:///home/yhlmaybe/Documents/Intelligent-Robot-System/RO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
- link LittleFingerArth_4_Link: geometry collision mesh filename=file:///home/yhlmaybe/Documents/Intelligent-Robot-System/RO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; visual mesh filename=file:///home/yhlmaybe/Documents/Intelligent-Robot-System/RO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
- link MidFingerArth_1_Link: geometry collision mesh filename=file:///home/yhlmaybe/Documents/Intelligent-Robot-System/RO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; visual mesh filename=file:///home/yhlmaybe/Documents/Intelligent-Robot-System/RO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
- link MidFingerArth_2_Link: geometry collision mesh filename=file:///home/yhlmaybe/Documents/Intelligent-Robot-System/RO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; visual mesh filename=file:///home/yhlmaybe/Documents/Intelligent-Robot-System/RO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
- link MidFingerArth_3_Link: geometry collision mesh filename=file:///home/yhlmaybe/Documents/Intelligent-Robot-System/RO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; visual mesh filename=file:///home/yhlmaybe/Documents/Intelligent-Robot-System/RO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
- link MidFingerArth_4_Link: geometry collision mesh filename=file:///home/yhlmaybe/Documents/Intelligent-Robot-System/RO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; visual mesh filename=file:///home/yhlmaybe/Documents/Intelligent-Robot-System/RO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
- link Palm_Link: geometry collision mesh filename=file:///home/yhlmaybe/Documents/Intelligent-Robot-System/RO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; visual mesh filename=file:///home/yhlmaybe/Documents/Intelligent-Robot-System/RO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
- link ThumbArth_1_Link: geometry collision mesh filename=file:///home/yhlmaybe/Documents/Intelligent-Robot-System/RO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; visual mesh filename=file:///home/yhlmaybe/Documents/Intelligent-Robot-System/RO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
- link ThumbArth_2_Link: geometry collision mesh filename=file:///home/yhlmaybe/Documents/Intelligent-Robot-System/RO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; visual mesh filename=file:///home/yhlmaybe/Documents/Intelligent-Robot-System/RO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
- link ThumbArth_3_Link: geometry collision mesh filename=file:///home/yhlmaybe/Documents/Intelligent-Robot-System/RO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; visual mesh filename=file:///home/yhlmaybe/Documents/Intelligent-Robot-System/RO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
- link ThumbArth_4_Link: geometry collision mesh filename=file:///home/yhlmaybe/Documents/Intelligent-Robot-System/RO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; visual mesh filename=file:///home/yhlmaybe/Documents/Intelligent-Robot-System/RO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
- link WristArth_Link: mass 0.00943638652052924 -> 0.0094364; geometry collision mesh filename=file:///home/yhlmaybe/Documents/Intelligent-Robot-System/RO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; visual mesh filename=file:///home/yhlmaybe/Documents/Intelligent-Robot-System/RO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
- link base_link: mass None -> 0.2802723579374; geometry collision mesh filename=file:///home/yhlmaybe/Documents/Intelligent-Robot-System/RO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; visual mesh filename=file:///home/yhlmaybe/Documents/Intelligent-Robot-System/RO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
Joints:
- joint FourthFingerArth_1_Joint: origin xyz=0 0.033328 0 rpy=0 0 0 -> xyz=0 0.0333280500386341 0 rpy=0 0 0
- joint FourthFingerArth_2_Joint: origin xyz=0 0.042169 0 rpy=0 0 0 -> xyz=0 0.0421689103147308 0 rpy=0 0 0
- joint FourthFingerArth_3_Joint: origin xyz=0 0.025759 0 rpy=0 0 0 -> xyz=0 0.025758853392147 0 rpy=0 0 0
- joint FourthFingerArth_4_Joint: origin xyz=0.015841 0.086236 -0.00256 rpy=0 0.22705 0 -> xyz=0.0158413525411462 0.0862362561371976 -0.00255995620301221 rpy=0 0.227050271472169 0
- joint IndexFingerArth_1_Joint: origin xyz=0 0.033328 0 rpy=0 0 0 -> xyz=0 0.0333280500386343 0 rpy=0 0 0
- joint IndexFingerArth_2_Joint: origin xyz=0 0.042169 0 rpy=0 0 0 -> xyz=0 0.0421689103147312 0 rpy=0 0 0
- joint IndexFingerArth_3_Joint: origin xyz=0 0.025759 0 rpy=0 0 0 -> xyz=0 0.025758853392147 0 rpy=0 0 0
- joint IndexFingerArth_4_Joint: origin xyz=-0.024616 0.088017 0.0042371 rpy=0 -0.016689 0 -> xyz=-0.0246155312110056 0.0880171234273368 0.00423706647925437 rpy=0 -0.016688636846923 0
- joint LittleFingerArth_1_Joint: origin xyz=0 0.033328 0 rpy=0 0 0 -> xyz=0 0.0333280500386338 0 rpy=0 0 0
- joint LittleFingerArth_2_Joint: axis -1 0 0 -> -0.974665262560157 -0.148230073829987 -0.167497675120869; origin xyz=0 0.033834 0 rpy=0 0 0 -> xyz=0 0.0338342375518586 0 rpy=0 0 0
- joint LittleFingerArth_3_Joint: axis -1 0 0 -> -0.97466526256011 -0.148230073829968 -0.167497675121158; origin xyz=0 0.025759 0 rpy=0 0 0 -> xyz=0 0.0257588533921475 0 rpy=0 0 0
- joint LittleFingerArth_4_Joint: origin xyz=0.038083 0.086957 -0.010175 rpy=-0.062663 0.3906 -0.16333 -> xyz=0.0380834548483633 0.0869571538128283 -0.0101752596541082 rpy=-0.0626625298576056 0.390601949010417 -0.163326502886668
- joint MidFingerArth_1_Joint: origin xyz=0 0.033328 0 rpy=0 0 0 -> xyz=0 0.0333280500386328 0 rpy=0 0 0
- joint MidFingerArth_2_Joint: origin xyz=0 0.0482 0 rpy=0 0 0 -> xyz=0 0.0481999999999999 0 rpy=0 0 0
- joint MidFingerArth_3_Joint: axis -1 0 0 -> -0.999685114570904 0 -0.0250932601580168; origin xyz=0 0.025759 0 rpy=0 0 0 -> xyz=0.0204834452846029 0.0257588533921481 0.00109576112089106 rpy=0 0.0250958943237956 0
- joint MidFingerArth_4_Joint: axis 0 0 1 -> 0.0250932601581999 0 0.999685114570899; origin xyz=-0.024616 0.088017 0.0042371 rpy=0 -0.016689 0 -> xyz=-0.0246155312110056 0.0880171234273368 0.00423706647925437 rpy=0 -0.016688636846923 0
- joint ThumbArth_1_Joint: origin xyz=0 0.033369 0 rpy=0 0 0 -> xyz=0 0.0333689103147325 0 rpy=0 0 0
- joint ThumbArth_2_Joint: origin xyz=0 0.048671 0 rpy=0 0 0 -> xyz=0 0.0486709159350182 0 rpy=0 0 0
- joint ThumbArth_3_Joint: origin xyz=0.00015994 0.0091836 0 rpy=3.1416 -1.5708 0 -> xyz=0.000159939498480935 0.00918364455238352 0 rpy=3.14159265358979 -1.5707963267949 0
- joint ThumbArth_4_Joint: origin xyz=-0.037378 0.02824 -0.010425 rpy=-0.017351 0.27783 1.5469 -> xyz=-0.0373776216869401 0.0282396610156985 -0.0104250544729608 rpy=-0.0173509972223506 0.277828062025534 1.54690272268651
- joint WristArth_Joint: origin xyz=0 0.0349997618236041 -0.0225000000000002 rpy=0 0 0 -> xyz=0 0.035 -0.0225 rpy=0 0 0

Commit message: update

File: ROSManager/urdf/Arm_R.SLDASM.urdf (robot description, URDF)
Before this commit: robot Arm_R.SLDASM, 23 links, 22 joints
Joints:
- joint FourthFingerArth_1_Joint: type continuous -> fixed
- joint FourthFingerArth_2_Joint: type continuous -> fixed
- joint FourthFingerArth_3_Joint: type continuous -> fixed
- joint FourthFingerArth_4_Joint: type continuous -> fixed
- joint IndexFingerArth_1_Joint: type continuous -> fixed
- joint IndexFingerArth_2_Joint: type continuous -> fixed
- joint IndexFingerArth_3_Joint: type continuous -> fixed
- joint IndexFingerArth_4_Joint: type continuous -> fixed
- joint LittleFingerArth_1_Joint: type continuous -> fixed
- joint LittleFingerArth_2_Joint: type continuous -> fixed
- joint LittleFingerArth_3_Joint: type continuous -> fixed
- joint LittleFingerArth_4_Joint: type continuous -> fixed
- joint MidFingerArth_1_Joint: type continuous -> fixed
- joint MidFingerArth_2_Joint: type continuous -> fixed
- joint MidFingerArth_3_Joint: type continuous -> fixed
- joint MidFingerArth_4_Joint: type continuous -> fixed
- joint Palm_Joint: type continuous -> fixed
- joint ThumbArth_1_Joint: type continuous -> fixed
- joint ThumbArth_2_Joint: type continuous -> fixed
- joint ThumbArth_3_Joint: type continuous -> fixed
- joint ThumbArth_4_Joint: origin xyz=-0.0373776216869401 0.0282396610156985 -0.0104250544729608 rpy=-0.0173509972223506 0.277828062025534 1.54690272268651 -> xyz=-0.037378 0.02824 -0.010425 rpy=-0.017351 0.27783 1.5469; type continuous -> fixed
- joint WristArth_Joint: type continuous -> fixed
