Commit message: update

File: Configure/Arm_R_SLDASM.urdf (robot description, URDF)
Before this commit: robot Arm_R_SLDASM, 23 links, 22 joints
Links:
- added link FourthEnd_Link, mass 0.000565670175158328; collision mesh filename=${URDF_MESH_PATH}/FourthEnd_Link.STL; visual mesh filename=${URDF_MESH_PATH}/FourthEnd_Link.STL
- added link IndexEnd_Link, mass 0.000565670175158323; collision mesh filename=${URDF_MESH_PATH}/IndexEnd_Link.STL; visual mesh filename=${URDF_MESH_PATH}/IndexEnd_Link.STL
- added link LittleEnd_Link, mass 0.000565670175158326; collision mesh filename=${URDF_MESH_PATH}/LittleEnd_Link.STL; visual mesh filename=${URDF_MESH_PATH}/LittleEnd_Link.STL
- added link MidEnd_Link, mass 0.000565670175158326; collision mesh filename=${URDF_MESH_PATH}/MidEnd_Link.STL; visual mesh filename=${URDF_MESH_PATH}/MidEnd_Link.STL
- added link ThumbEnd_Link, mass 0.000597070725003369; collision mesh filename=${URDF_MESH_PATH}/ThumbEnd_Link.STL; visual mesh filename=${URDF_MESH_PATH}/ThumbEnd_Link.STL
- link FourthFingerArth_1_Link: geometry collision mesh filename=${URDF_MESH_PATH}/FourthFingerArth_1_Link.STL; visual mesh filename=${URDF_MESH_PATH}/FourthFingerArth_1_Link.STL
- link FourthFingerArth_2_Link: geometry collision mesh filename=${URDF_MESH_PATH}/FourthFingerArth_2_Link.STL; visual mesh filename=${URDF_MESH_PATH}/FourthFingerArth_2_Link.STL
- link FourthFingerArth_3_Link: mass 0.0013727 -> 0.00137270637615468; geometry collision mesh filename=${URDF_MESH_PATH}/FourthFingerArth_3_Link.STL; visual mesh filename=${URDF_MESH_PATH}/FourthFingerArth_3_Link.STL
- link FourthFingerArth_4_Link: geometry collision mesh filename=${URDF_MESH_PATH}/FourthFingerArth_4_Link.STL; visual mesh filename=${URDF_MESH_PATH}/FourthFingerArth_4_Link.STL
- link IndexFingerArth_1_Link: geometry collision mesh filename=${URDF_MESH_PATH}/IndexFingerArth_1_Link.STL; visual mesh filename=${URDF_MESH_PATH}/IndexFingerArth_1_Link.STL
- link IndexFingerArth_2__Link: geometry collision mesh filename=${URDF_MESH_PATH}/IndexFingerArth_2__Link.STL; visual mesh filename=${URDF_MESH_PATH}/IndexFingerArth_2__Link.STL
- link IndexFingerArth_3_Link: geometry collision mesh filename=${URDF_MESH_PATH}/IndexFingerArth_3_Link.STL; visual mesh filename=${URDF_MESH_PATH}/IndexFingerArth_3_Link.STL
- link IndexFingerArth_4_Link: geometry collision mesh filename=${URDF_MESH_PATH}/IndexFingerArth_4_Link.STL; visual mesh filename=${URDF_MESH_PATH}/IndexFingerArth_4_Link.STL
- link LittleFingerArth_1_Link: geometry collision mesh filename=${URDF_MESH_PATH}/LittleFingerArth_1_Link.STL; visual mesh filename=${URDF_MESH_PATH}/LittleFingerArth_1_Link.STL
- link LittleFingerArth_2_Link: geometry collision mesh filename=${URDF_MESH_PATH}/LittleFingerArth_2_Link.STL; visual mesh filename=${URDF_MESH_PATH}/LittleFingerArth_2_Link.STL
- link LittleFingerArth_3_Link: geometry collision mesh filename=${URDF_MESH_PATH}/LittleFingerArth_3_Link.STL; visual mesh filename=${URDF_MESH_PATH}/LittleFingerArth_3_Link.STL
- link LittleFingerArth_4_Link: mass 0.0024833 -> 0.00248334722292415; geometry collision mesh filename=${URDF_MESH_PATH}/LittleFingerArth_4_Link.STL; visual mesh filename=${URDF_MESH_PATH}/LittleFingerArth_4_Link.STL
- link MidFingerArth_1_Link: geometry collision mesh filename=${URDF_MESH_PATH}/MidFingerArth_1_Link.STL; visual mesh filename=${URDF_MESH_PATH}/MidFingerArth_1_Link.STL
- link MidFingerArth_2_Link: geometry collision mesh filename=${URDF_MESH_PATH}/MidFingerArth_2_Link.STL; visual mesh filename=${URDF_MESH_PATH}/MidFingerArth_2_Link.STL
- link MidFingerArth_3_Link: mass 0.0015967 -> 0.00159667671601455; geometry collision mesh filename=${URDF_MESH_PATH}/MidFingerArth_3_Link.STL; visual mesh filename=${URDF_MESH_PATH}/MidFingerArth_3_Link.STL
- link MidFingerArth_4_Link: geometry collision mesh filename=${URDF_MESH_PATH}/MidFingerArth_4_Link.STL; visual mesh filename=${URDF_MESH_PATH}/MidFingerArth_4_Link.STL
- link Palm_Link: mass 0.043011 -> 0.043010605375804; geometry collision mesh filename=${URDF_MESH_PATH}/Palm_Link.STL; visual mesh filename=${URDF_MESH_PATH}/Palm_Link.STL
- link ThumbArth_1_Link: geometry collision mesh filename=${URDF_MESH_PATH}/ThumbArth_1_Link.STL; visual mesh filename=${URDF_MESH_PATH}/ThumbArth_1_Link.STL
- link ThumbArth_2_Link: geometry collision mesh filename=${URDF_MESH_PATH}/ThumbArth_2_Link.STL; visual mesh filename=${URDF_MESH_PATH}/ThumbArth_2_Link.STL
- link ThumbArth_3_Link: mass 0.0027656 -> 0.00276558683424971; geometry collision mesh filename=${URDF_MESH_PATH}/ThumbArth_3_Link.STL; visual mesh filename=${URDF_MESH_PATH}/ThumbArth_3_Link.STL
- link ThumbArth_4_Link: geometry collision mesh filename=${URDF_MESH_PATH}/ThumbArth_4_Link.STL; visual mesh filename=${URDF_MESH_PATH}/ThumbArth_4_Link.STL
- link WristArth_Link: geometry collision mesh filename=${URDF_MESH_PATH}/WristArth_Link.STL; visual mesh filename=${URDF_MESH_PATH}/WristArth_Link.STL
- link base_link: mass 0.28027 -> 0.2802723579374; geometry collision mesh filename=${URDF_MESH_PATH}/base_link.STL; visual mesh filename=${URDF_MESH_PATH}/base_link.STL
Joints:
- added joint FourthEnd_Joint: type fixed, parent FourthFingerArth_1_Link, child FourthEnd_Link, origin xyz=0.0190841404860265 0.001943926716239 0 rpy=0 0 0, axis 0 0 0
- added joint IndexEnd_Joint: type fixed, parent IndexFingerArth_1_Link, child IndexEnd_Link, origin xyz=0.0190841404860254 0.00194392671623844 0 rpy=0 0 0, axis 0 0 0
- added joint LittleEnd_Joint: type fixed, parent LittleFingerArth_1_Link, child LittleEnd_Link, origin xyz=0.0190841404860253 0.00194392671623847 0 rpy=0 0 0, axis 0 0 0
- added joint MidEnd_Joint: type fixed, parent MidFingerArth_1_Link, child MidEnd_Link, origin xyz=0.0190841404860259 0.001943926716239 0 rpy=0 0 0, axis 0 0 0
- added joint ThumbEnd_Join: type fixed, parent ThumbArth_1_Link, child ThumbEnd_Link, origin xyz=0.023781 0.0016665 0 rpy=0 0 0, axis 0 0 0
- joint FourthFingerArth_1_Joint: origin xyz=0.033328 0 0 rpy=0 0 0 -> xyz=0.0333280500386341 0 0 rpy=0 0 0; type continuous -> revolute
- joint FourthFingerArth_2_Joint: origin xyz=0.042169 0 0 rpy=0 0 0 -> xyz=0.0421689103147308 0 0 rpy=0 0 0; type continuous -> revolute
- joint FourthFingerArth_3_Joint: origin xyz=0 0.025759 0 rpy=-1.5708 0 1.5708 -> xyz=0 0.025758853392147 0 rpy=-1.5707963267949 0 1.57079632679491; type continuous -> revolute
- joint FourthFingerArth_4_Joint: origin xyz=0.00256 0.086236 0.015841 rpy=0 -1.3437 0 -> xyz=0.00255995620301201 0.0862362561371976 0.0158413525411461 rpy=0 -1.34374605532273 0; type continuous -> revolute
- joint IndexFingerArth_1_Joint: origin xyz=0.033328 0 0 rpy=0 0 0 -> xyz=0.0333280500386343 0 0 rpy=0 0 0; type continuous -> revolute
- joint IndexFingerArth_2_Joint: origin xyz=0.042169 0 0 rpy=0 0 0 -> xyz=0.0421689103147312 0 0 rpy=0 0 0; type continuous -> revolute
- joint IndexFingerArth_3_Joint: type continuous -> revolute
- joint IndexFingerArth_4_Joint: type continuous -> revolute
- joint LittleFingerArth_1_Joint: origin xyz=0.033328 0 0 rpy=0 0 0 -> xyz=0.0333280500386338 0 0 rpy=0 0 0; type continuous -> revolute
- joint LittleFingerArth_2_Joint: origin xyz=0.033834 0 0 rpy=0 0 0 -> xyz=0.0338342375518586 0 0 rpy=0 0 0; type continuous -> revolute
- joint LittleFingerArth_3_Joint: origin xyz=0 0.025759 0 rpy=-1.5708 0 1.5708 -> xyz=0 0.0257588533921475 0 rpy=-1.57079632679514 0 1.5707963267949; type continuous -> revolute
- joint LittleFingerArth_4_Joint: origin xyz=0.010175 0.086957 0.038083 rpy=0.34581 -1.149 -0.3761 -> xyz=0.010175259654108 0.0869571538128283 0.0380834548483633 rpy=0.345813814936415 -1.14904704904316 -0.37609749493507; type continuous -> revolute
- joint MidFingerArth_1_Joint: origin xyz=0.033328 0 0 rpy=0 0 0 -> xyz=0.0333280500386328 0 0 rpy=0 0 0; type continuous -> revolute
- joint MidFingerArth_2_Joint: origin xyz=0.0482 0 0 rpy=0 0 0 -> xyz=0.0481999999999999 0 0 rpy=0 0 0; type continuous -> revolute
- joint MidFingerArth_3_Joint: origin xyz=0 0.025759 0 rpy=-1.5708 0 1.5708 -> xyz=0 0.0257588533921476 0 rpy=-1.57079632679508 0 1.5707963267949; type continuous -> revolute
- joint MidFingerArth_4_Joint: origin xyz=-0.0056745 0.088017 -0.0041532 rpy=0 -1.5624 0 -> xyz=-0.00567449992537894 0.0880171234273373 -0.00415322419910361 rpy=0 -1.56238906931784 0; type continuous -> revolute
- joint Palm_Joint: type continuous -> revolute
- joint ThumbArth_1_Joint: origin xyz=0.033369 0 0 rpy=0 0 0.0029994 -> xyz=0.033369 0 0 rpy=0 0 0; type continuous -> revolute
- joint ThumbArth_2_Joint: origin xyz=-0.048671 0 0 rpy=0 0 3.1416 -> xyz=0.048671 0 0 rpy=0 0 0; type continuous -> revolute
- joint ThumbArth_3_Joint: limit lower=0 upper=1.5708 effort=1.67 velocity=7.48 -> lower=-1.5708 upper=0 effort=1.67 velocity=7.48; origin xyz=0 0.0091836 -0.00015994 rpy=1.5708 0 -1.5708 -> xyz=0 0.0091836 -0.00015994 rpy=-1.5708 0 1.5708; type continuous -> revolute
- joint ThumbArth_4_Joint: limit lower=-0.174533 upper=2.967061 effort=1.67 velocity=7.48 -> lower=0 upper=3.1416 effort=1.67 velocity=7.48; type continuous -> revolute
- joint WristArth_Joint: type continuous -> revolute

Commit message: update

File: Configure/Arm_R_SLDASM.urdf (robot description, URDF)
Before this commit: robot Arm_R_SLDASM, 28 links, 27 joints
Links:
- link FourthEnd_Link: geometry collision mesh filename=${URDF_COLLISION_MESH_PATH}/FourthEnd_Link.STL; visual mesh filename=${URDF_VISUAL_MESH_PATH}/FourthEnd_Link.STL
- link FourthFingerArth_1_Link: geometry collision mesh filename=${URDF_COLLISION_MESH_PATH}/FourthFingerArth_1_Link.STL; visual mesh filename=${URDF_VISUAL_MESH_PATH}/FourthFingerArth_1_Link.STL
- link FourthFingerArth_2_Link: geometry collision mesh filename=${URDF_COLLISION_MESH_PATH}/FourthFingerArth_2_Link.STL; visual mesh filename=${URDF_VISUAL_MESH_PATH}/FourthFingerArth_2_Link.STL
- link FourthFingerArth_3_Link: geometry collision mesh filename=${URDF_COLLISION_MESH_PATH}/FourthFingerArth_3_Link.STL; visual mesh filename=${URDF_VISUAL_MESH_PATH}/FourthFingerArth_3_Link.STL
- link FourthFingerArth_4_Link: geometry collision mesh filename=${URDF_COLLISION_MESH_PATH}/FourthFingerArth_4_Link.STL; visual mesh filename=${URDF_VISUAL_MESH_PATH}/FourthFingerArth_4_Link.STL
- link IndexEnd_Link: geometry collision mesh filename=${URDF_COLLISION_MESH_PATH}/IndexEnd_Link.STL; visual mesh filename=${URDF_VISUAL_MESH_PATH}/IndexEnd_Link.STL
- link IndexFingerArth_1_Link: geometry collision mesh filename=${URDF_COLLISION_MESH_PATH}/IndexFingerArth_1_Link.STL; visual mesh filename=${URDF_VISUAL_MESH_PATH}/IndexFingerArth_1_Link.STL
- link IndexFingerArth_2__Link: geometry collision mesh filename=${URDF_COLLISION_MESH_PATH}/IndexFingerArth_2__Link.STL; visual mesh filename=${URDF_VISUAL_MESH_PATH}/IndexFingerArth_2__Link.STL
- link IndexFingerArth_3_Link: geometry collision mesh filename=${URDF_COLLISION_MESH_PATH}/IndexFingerArth_3_Link.STL; visual mesh filename=${URDF_VISUAL_MESH_PATH}/IndexFingerArth_3_Link.STL
- link IndexFingerArth_4_Link: geometry collision mesh filename=${URDF_COLLISION_MESH_PATH}/IndexFingerArth_4_Link.STL; visual mesh filename=${URDF_VISUAL_MESH_PATH}/IndexFingerArth_4_Link.STL
- link LittleEnd_Link: geometry collision mesh filename=${URDF_COLLISION_MESH_PATH}/LittleEnd_Link.STL; visual mesh filename=${URDF_VISUAL_MESH_PATH}/LittleEnd_Link.STL
- link LittleFingerArth_1_Link: geometry collision mesh filename=${URDF_COLLISION_MESH_PATH}/LittleFingerArth_1_Link.STL; visual mesh filename=${URDF_VISUAL_MESH_PATH}/LittleFingerArth_1_Link.STL
- link LittleFingerArth_2_Link: geometry collision mesh filename=${URDF_COLLISION_MESH_PATH}/LittleFingerArth_2_Link.STL; visual mesh filename=${URDF_VISUAL_MESH_PATH}/LittleFingerArth_2_Link.STL
- link LittleFingerArth_3_Link: geometry collision mesh filename=${URDF_COLLISION_MESH_PATH}/LittleFingerArth_3_Link.STL; visual mesh filename=${URDF_VISUAL_MESH_PATH}/LittleFingerArth_3_Link.STL
- link LittleFingerArth_4_Link: geometry collision mesh filename=${URDF_COLLISION_MESH_PATH}/LittleFingerArth_4_Link.STL; visual mesh filename=${URDF_VISUAL_MESH_PATH}/LittleFingerArth_4_Link.STL
- link MidEnd_Link: geometry collision mesh filename=${URDF_COLLISION_MESH_PATH}/MidEnd_Link.STL; visual mesh filename=${URDF_VISUAL_MESH_PATH}/MidEnd_Link.STL
- link MidFingerArth_1_Link: geometry collision mesh filename=${URDF_COLLISION_MESH_PATH}/MidFingerArth_1_Link.STL; visual mesh filename=${URDF_VISUAL_MESH_PATH}/MidFingerArth_1_Link.STL
- link MidFingerArth_2_Link: geometry collision mesh filename=${URDF_COLLISION_MESH_PATH}/MidFingerArth_2_Link.STL; visual mesh filename=${URDF_VISUAL_MESH_PATH}/MidFingerArth_2_Link.STL
- link MidFingerArth_3_Link: geometry collision mesh filename=${URDF_COLLISION_MESH_PATH}/MidFingerArth_3_Link.STL; visual mesh filename=${URDF_VISUAL_MESH_PATH}/MidFingerArth_3_Link.STL
- link MidFingerArth_4_Link: geometry collision mesh filename=${URDF_COLLISION_MESH_PATH}/MidFingerArth_4_Link.STL; visual mesh filename=${URDF_VISUAL_MESH_PATH}/MidFingerArth_4_Link.STL
- link Palm_Link: geometry collision mesh filename=${URDF_COLLISION_MESH_PATH}/Palm_Link.STL; visual mesh filename=${URDF_VISUAL_MESH_PATH}/Palm_Link.STL
- link ThumbArth_1_Link: geometry collision mesh filename=${URDF_COLLISION_MESH_PATH}/ThumbArth_1_Link.STL; visual mesh filename=${URDF_VISUAL_MESH_PATH}/ThumbArth_1_Link.STL
- link ThumbArth_2_Link: geometry collision mesh filename=${URDF_COLLISION_MESH_PATH}/ThumbArth_2_Link.STL; visual mesh filename=${URDF_VISUAL_MESH_PATH}/ThumbArth_2_Link.STL
- link ThumbArth_3_Link: geometry collision mesh filename=${URDF_COLLISION_MESH_PATH}/ThumbArth_3_Link.STL; visual mesh filename=${URDF_VISUAL_MESH_PATH}/ThumbArth_3_Link.STL
- link ThumbArth_4_Link: geometry collision mesh filename=${URDF_COLLISION_MESH_PATH}/ThumbArth_4_Link.STL; visual mesh filename=${URDF_VISUAL_MESH_PATH}/ThumbArth_4_Link.STL
- link ThumbEnd_Link: geometry collision mesh filename=${URDF_COLLISION_MESH_PATH}/ThumbEnd_Link.STL; visual mesh filename=${URDF_VISUAL_MESH_PATH}/ThumbEnd_Link.STL
- link WristArth_Link: geometry collision mesh filename=${URDF_COLLISION_MESH_PATH}/WristArth_Link.STL; visual mesh filename=${URDF_VISUAL_MESH_PATH}/WristArth_Link.STL
- link base_link: geometry collision mesh filename=${URDF_COLLISION_MESH_PATH}/base_link.STL; visual mesh filename=${URDF_VISUAL_MESH_PATH}/base_link.STL
